Commit message: Added simulation_launch. Other people can clone the repository, build it, then run it right away

File: simulation_launch/models/alphabot2/model.urdf (robot description, URDF)
Before this commit: robot mobile_bot, 7 links, 6 joints
Links:
- removed link drivewhl_l_link
- removed link drivewhl_r_link
- removed link front_caster
- added link caster_wheel_b_link, mass 2; collision sphere radius=0.035; visual sphere radius=0.035
- added link caster_wheel_f_link, mass 2; collision sphere radius=0.035; visual sphere radius=0.035
- added link drive_wheel_l_link, mass 2; collision cylinder length=0.04 radius=0.07; visual cylinder length=0.04 radius=0.07
- added link drive_wheel_r_link, mass 2; collision cylinder length=0.04 radius=0.07; visual cylinder length=0.04 radius=0.07
- link base_link: geometry collision cylinder length=0.3 radius=0.2; visual cylinder length=0.3 radius=0.2
- link lidar_link: mass 0.125 -> 0.1; geometry collision cylinder length=0.07 radius=0.1; visual cylinder length=0.07 radius=0.1
Joints:
- removed joint caster_joint
- removed joint drivewhl_l_joint
- removed joint drivewhl_r_joint
- added joint caster_wheel_b_joint: type fixed, parent base_link, child caster_wheel_b_link, origin xyz=-0.165 0 -0.155 rpy=0 0 0
- added joint caster_wheel_f_joint: type fixed, parent base_link, child caster_wheel_f_link, origin xyz=0.165 0 -0.155 rpy=0 0 0
- added joint drive_wheel_l_joint: type continuous, parent base_link, child drive_wheel_l_link, origin xyz=0 0.22 -0.12 rpy=0 0 0, axis 0 1 0
- added joint drive_wheel_r_joint: type continuous, parent base_link, child drive_wheel_r_link, origin xyz=0 -0.22 -0.12 rpy=0 0 0, axis 0 1 0
- joint base_joint: origin xyz=0 0 0.15000000000000002 rpy=0 0 0 -> xyz=0 0 0.19 rpy=0 0 0
- joint imu_joint: origin xyz=0 0 0.01 -> xyz=0 0 0
- joint lidar_joint: origin xyz=0 0 0.12 rpy=0 0 0 -> xyz=0 0 0.185 rpy=0 0 0
